File: opto_staccato_controller/opto_staccato_controller.kicad_sch (KiCad schematic)
At the start: 60 parts, among them J1 120/240VAC, J2 External Signal, J5 Jumper, J6 Jumper, Q1 2N3906, Q2 2N3904, Q3 2N3904, SW1 SW_SPDT, SW2 SW_SPDT, SW3 SW_SP3T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

Commit message: Add license to source files and images of schematics
Other:
- note added: "Copyright Nick Ohi, Coil Labs 2022. This source describes Open Hardware and is licensed under the CERN-OHL- W v2 You may redistribute and modify this documentation and make products using it under the terms of the CERN-OHL-W v2 (https:/cern.ch/cern-ohl). This documentation is distributed WITHOUT ANY EXPRESS OR IMPLIED WARRANTY, INCLUDING OF MERCHANTABILITY, SATISFACTORY QUALITY AND FITNESS FOR A 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"
Changed lines of the file:
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@@
     (stroke (width 0) (type default) (color 0 0 0 0))
   )
-  (text "All resistors are 1/2W unless otherwise indicated" (at 302.26 257.81 0)
+  (text "All resistors are 1/2W unless otherwise indicated" (at 144.78 139.7 0)
     (effects (font (size 1.27 1.27)) (justify left bottom))
   )
+  (text "Copyright Nick Ohi, Coil Labs 2022.\nThis source describes Open Hardware and is licensed under the CERN-OHL-\nW v2\nYou may redistribute and modify this documentation and make products\nusing it under the terms of the CERN-OHL-W v2 (https:/cern.ch/cern-ohl).\nThis documentation is distributed WITHOUT ANY EXPRESS OR IMPLIED\nWARRANTY, INCLUDING OF MERCHANTABILITY, SATISFACTORY QUALITY\nAND FITNESS FOR A PARTICULAR PURPOSE. Please see the CERN-OHL-W v2\nfor applicable conditions.\nSource location: https://github.com/Coil-Labs/opto-staccato"
+    (at 269.24 154.94 0)
+    (effects (font (size 1.27 1.27)) (justify left bottom))
+  )
